File: Arduino/Ard-perf++.sch (KiCad schematic (older format))
At the start: 8 parts, among them P1 Power, P2 Analog, P3 Digital, P4 Digital, P5 CONN_01X01, P6 CONN_01X01, P7 CONN_01X01, P8 CONN_01X01

Commit message: updates and name consistency to Ard
Connections:
- net labels added: GND3
- wire segments 114 -> 112
Changed lines of the file:
@@
 Wire Wire Line
 	9400 2200 9300 2200
-Connection ~ 9300 2200
 Wire Wire Line
 	8950 2300 8950 1450
@@
 Wire Wire Line
 	10300 1500 10300 3150
-Wire Wire Line
-	9300 2100 9300 3150
 Wire Notes Line
 	8700 1000 11200 1000
@@
 	5350 3150 5700 3150
 Wire Wire Line
-	5350 3300 5500 3300
-Wire Wire Line
-	5500 3300 5500 3150
-Connection ~ 5500 3150
+	5350 3300 5700 3300
 Wire Wire Line
 	5700 3000 5350 3000
@@
 Text Label 5550 3000 0    60   ~ 0
 5V
-Text Label 9300 3150 0    60   ~ 0
+Text Label 9300 2100 2    60   ~ 0
 GND1
 Text Label 10300 3150 0    60   ~ 0
@@
 Text Label 1250 3000 2    60   ~ 0
 GND2
+Text Label 5550 3300 0    60   ~ 0
+GND3
+Text Label 9300 2200 2    60   ~ 0
+GND3
 $EndSCHEMATC
