File: Arduino/Ard-perf++.kicad_pcb (KiCad board)
At the start: 2 copper layers, 68.6 x 53.3 mm, 457 parts, among them P1 Power, P2 Analog, P3 Digital, P4 Digital, P5 CONN_01X01, P6 CONN_01X01, P7 CONN_01X01, P8 CONN_01X01

Commit message: updates and name consistency to Ard
Connections:
- JR17 pad 1: /15x25perf2/JR16 -> /15x25perf2/JR17
- P1 pad 7: /15x25perf2/JR16 -> /15x25perf2/JR17
Routing:
- net /15x25perf2/JR16: track 7.62 -> 2.54 mm
- net /15x25perf2/JR17: track 0.00 -> 2.54 mm
Other:
- board text added: "Ard-Perf++"
- board text removed: "Ard-Perf+2"
Changed lines of the file:
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@@
 (kicad_pcb (version 4) (host pcbnew 4.0.2-stable)
   (general
-    (links 887)
+    (links 886)
     (no_connects 0)
-    (area 110.922999 71.582 374.447405 127.404)
+    (area 110.922999 72.949999 179.653001 126.440001)
     (thickness 1.6)
-    (drawings 150)
-    (tracks 932)
+    (drawings 155)
+    (tracks 931)
     (zones 0)
     (modules 457)
-    (nets 497)
+    (nets 498)
   )
   (page A4)
@@
     (visible_elements 7FFFFFFF)
     (pcbplotparams
-      (layerselection 0x00030_80000001)
+      (layerselection 0x010f0_80000001)
       (usegerberextensions false)
       (excludeedgelayer true)
@@
       (outputformat 1)
       (mirror false)
-      (drillshape 1)
+      (drillshape 0)
       (scaleselection 1)
-      (outputdirectory ""))
+      (outputdirectory gerbers/))
   )
   (net 0 "")
@@
   (net 495 "Net-(JJ25-Pad1)")
   (net 496 "Net-(JJ26-Pad1)")
+  (net 497 /15x25perf2/JR17)
   (net_class Default "This is the default net class."
     (clearance 0.01)
@@
     (add_net /15x25perf2/JR13)
     (add_net /15x25perf2/JR16)
+    (add_net /15x25perf2/JR17)
     (add_net /15x25perf2/JR18)
     (add_net /15x25perf2/JR20)
@@
       (net 467 /15x25perf2/JR16))
     (pad 7 thru_hole oval (at 15.24 0) (size 1.7272 2.032) (drill 1.016) (layers *.Cu *.Mask F.SilkS)
-      (net 467 /15x25perf2/JR16))
+      (net 497 /15x25perf2/JR17))
     (pad 8 thru_hole oval (at 17.78 0) (size 1.7272 2.032) (drill 1.016) (layers *.Cu *.Mask F.SilkS)
       (net 460 /15x25perf2/JR18))
@@
       (net 35 /15x25perf/J17))
     (pad 1 thru_hole circle (at 0 0 180) (size 1.4478 1.4478) (drill 1.0922) (layers *.Cu *.Mask)
-      (net 467 /15x25perf2/JR16))
+      (net 497 /15x25perf2/JR17))
     (pad 3 smd rect (at 0 1.143 270) (size 0.508 1.524) (layers B.Cu B.Mask)
       (net 449 /15x25perf2/JR))
@@
       (net 9 /15x25perf/JA))
   )
+  (gr_text "Rev A" (at 114.554 124.333) (layer B.SilkS)
+    (effects (font (size 1.27 1.27) (thickness 0.3)) (justify mirror))
+  )
+  (gr_text Inc. (at 120.65 124.333) (layer B.SilkS)
+    (effects (font (size 1.27 1.27) (thickness 0.254)) (justify mirror))
+  )
+  (gr_text "Fyber Labs" (at 132.334 124.333) (layer B.SilkS)
+    (effects (font (size 1.27 1.27) (thickness 0.254)) (justify mirror))
+  )
+  (gr_text 25 (at 174.498 114.808) (layer B.SilkS)
+    (effects (font (size 0.508 0.508) (thickness 0.127)) (justify mirror))
+  )
+  (gr_text Ard-Perf++ (at 117.094 74.549) (layer B.SilkS)
+    (effects (font (size 1.27 1.27) (thickness 0.3)) (justify mirror))
+  )
   (gr_line (start 174.498 78.105) (end 174.498 75.565) (layer B.SilkS) (width 1.75))
   (gr_line (start 171.958 78.105) (end 171.958 75.565) (layer B.SilkS) (width 1.75))
@@
     (effects (font (size 1.27 1.27) (thickness 0.3)))
   )
-  (gr_text Ard-Perf+2 (at 117.348 74.549) (layer F.SilkS)
+  (gr_text Ard-Perf++ (at 117.348 74.549) (layer F.SilkS)
     (effects (font (size 1.27 1.27) (thickness 0.3)))
   )
@@
   (segment (start 136.398 76.581) (end 136.398 78.105) (width 0.508) (layer F.Cu) (net 466))
   (segment (start 137.414 75.565) (end 136.398 76.581) (width 0.508) (layer F.Cu) (net 466))
-  (segment (start 154.178 123.825) (end 154.178 121.285) (width 0.508) (layer B.Cu) (net 467))
   (segment (start 151.638 123.825) (end 151.638 121.285) (width 0.508) (layer B.Cu) (net 467))
-  (segment (start 151.638 123.825) (end 154.178 123.825) (width 0.508) (layer F.Cu) (net 467))
   (segment (start 171.958 123.825) (end 171.958 121.285) (width 0.508) (layer B.Cu) (net 468))
   (segment (start 174.498 123.825) (end 174.498 121.285) (width 0.508) (layer B.Cu) (net 469))
@@
   (segment (start 171.958 99.822) (end 174.498 99.822) (width 0.508) (layer B.Cu) (net 471))
   (segment (start 174.498 99.822) (end 177.038 99.822) (width 0.508) (layer B.Cu) (net 471))
+  (segment (start 154.178 123.825) (end 154.178 121.285) (width 0.508) (layer B.Cu) (net 497))
 )

Commit message: edit tight corner
Routing:
- net /15x25perf/J25: track 45.3 -> 46.2 mm
Changed lines of the file:
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@@
     (thickness 1.6)
     (drawings 155)
-    (tracks 931)
+    (tracks 934)
     (zones 0)
     (modules 457)
@@
     (mod_text_size 1 1)
     (mod_text_width 0.15)
-    (pad_size 4.064 4.064)
-    (pad_drill 3.048)
+    (pad_size 0.508 1.4605)
+    (pad_drill 0)
     (pad_to_mask_clearance 0)
     (aux_axis_origin 110.998 126.365)
@@
     (fp_line (start -0.6096 -0.6858) (end 0 -0.635) (layer F.Cu) (width 0.1778))
     (fp_line (start -0.635 0) (end -0.6096 -0.6858) (layer F.Cu) (width 0.1778))
-    (pad 2 smd rect (at -1.143 0 180) (size 0.508 1.524) (layers F.Cu F.Mask)
+    (pad 2 smd rect (at -1.143 -0.0762 180) (size 0.508 1.4605) (layers F.Cu F.Mask)
       (net 51 /15x25perf/J25))
     (pad 1 thru_hole circle (at 0 0 180) (size 1.4478 1.4478) (drill 1.0922) (layers *.Cu *.Mask)
@@
   (segment (start 173.101 118.745) (end 173.101 121.285) (width 0.508) (layer F.Cu) (net 49))
   (segment (start 171.958 75.565) (end 171.958 78.105) (width 0.508) (layer F.Cu) (net 50))
+  (segment (start 175.641 113.665) (end 175.641 115.2231) (width 0.508) (layer F.Cu) (net 51))
+  (segment (start 175.641 115.2231) (end 174.3456 116.5185) (width 0.508) (layer F.Cu) (net 51))
+  (segment (start 174.3456 116.5185) (end 174.3456 119.507) (width 0.508) (layer F.Cu) (net 51))
+  (segment (start 174.3456 119.507) (end 174.92218 120.08358) (width 0.508) (layer F.Cu) (net 51))
+  (segment (start 174.3456 119.5578) (end 174.5615 119.5578) (width 0.254) (layer F.Cu) (net 51))
+  (segment (start 174.5615 119.5578) (end 175.641 120.6373) (width 0.254) (layer F.Cu) (net 51))
+  (segment (start 175.641 120.6373) (end 175.641 120.8532) (width 0.254) (layer F.Cu) (net 51))
   (segment (start 175.641 85.725) (end 175.641 87.2831) (width 0.508) (layer F.Cu) (net 51))
   (segment (start 175.641 87.2831) (end 174.3964 88.5277) (width 0.508) (layer F.Cu) (net 51))
@@
   (segment (start 174.3964 92.0115) (end 175.641 93.2561) (width 0.508) (layer F.Cu) (net 51))
   (segment (start 175.641 93.2561) (end 175.641 95.885) (width 0.508) (layer F.Cu) (net 51))
-  (segment (start 175.641 113.665) (end 175.641 115.2231) (width 0.508) (layer F.Cu) (net 51))
-  (segment (start 175.641 115.2231) (end 174.3456 116.5185) (width 0.508) (layer F.Cu) (net 51))
-  (segment (start 174.3456 116.5185) (end 174.3456 119.5578) (width 0.508) (layer F.Cu) (net 51))
-  (segment (start 174.3456 119.5578) (end 175.641 120.8532) (width 0.508) (layer F.Cu) (net 51))
   (segment (start 175.641 120.8532) (end 175.641 121.285) (width 0.508) (layer F.Cu) (net 51))
   (segment (start 175.641 78.105) (end 175.641 80.645) (width 0.508) (layer F.Cu) (net 51))
